File: BMS/BalanceSenseBlock.kicad_sch (KiCad schematic)
At the start: 7 parts, among them Q2 BSS308PE

Commit message: BMS Schema Done!
hello world
Parts:
- C5: renamed from C4; footprint Capacitor_SMD:C_0805_2012Metric_Pad1.15x1.40mm_HandSolder -> Capacitor_SMD:C_0805_2012Metric_Pad1.18x1.45mm_HandSolder
- R15: renamed from R9; footprint Resistor_SMD:R_0805_2012Metric_Pad1.15x1.40mm_HandSolder -> Resistor_SMD:R_0805_2012Metric_Pad1.20x1.40mm_HandSolder
- R16: renamed from R10; footprint Resistor_SMD:R_2512_6332Metric_Pad1.52x3.35mm_HandSolder -> Resistor_SMD:R_2512_6332Metric_Pad1.40x3.35mm_HandSolder
- R17: renamed from R11; footprint Resistor_SMD:R_0805_2012Metric_Pad1.15x1.40mm_HandSolder -> Resistor_SMD:R_0805_2012Metric_Pad1.20x1.40mm_HandSolder
- R18: renamed from R14; footprint Resistor_SMD:R_0805_2012Metric_Pad1.15x1.40mm_HandSolder -> Resistor_SMD:R_0805_2012Metric_Pad1.20x1.40mm_HandSolder
- renumbered D2 to D3, Q2 to Q3
Changed lines of the file:
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@@
 	(paper "A4")
+	(junction
+		(at 156.21 57.15)
+		(diameter 0)
+		(color 0 0 0 0)
+	)
+	(junction
+		(at 121.92 74.93)
+		(diameter 0)
+		(color 0 0 0 0)
+	)
+	(junction
+		(at 109.22 83.82)
+		(diameter 0)
+		(color 0 0 0 0)
+	)
 	(junction
 		(at 121.92 57.15)
@@
 		(color 0 0 0 0)
 	)
-	(junction
-		(at 156.21 57.15)
-		(diameter 0)
-		(color 0 0 0 0)
-	)
-	(junction
-		(at 121.92 74.93)
-		(diameter 0)
-		(color 0 0 0 0)
-	)
-	(junction
-		(at 109.22 83.82)
-		(diameter 0)
-		(color 0 0 0 0)
-	)
 	(polyline
 		(pts
@@
 	(wire
 		(pts
+			(xy 121.92 57.15) (xy 130.81 57.15)
+		)
+		(stroke
+			(width 0)
+			(type default)
+		)
+	)
+	(wire
+		(pts
 			(xy 156.21 57.15) (xy 156.21 66.04)
 		)
@@
 		(pts
 			(xy 156.21 77.47) (xy 165.1 77.47)
-		)
-		(stroke
-			(width 0)
-			(type default)
-		)
-	)
-	(wire
-		(pts
-			(xy 121.92 57.15) (xy 130.81 57.15)
 		)
 		(stroke
@@
 		(on_board yes)
 		(dnp no)
-		(property "Reference" "Q2"
+		(property "Reference" "Q3"
 			(at 119.2276 68.6816 0)
 			(effects
@@
 		(instances
 			(project ""
-				(path "/dc0b64a3-156e-446d-a433-c56b0c761cf1/00000000-0000-0000-0000-00005f7bc591"
-					(reference "Q2")
-					(unit 1)
-				)
 				(path "/dc0b64a3-156e-446d-a433-c56b0c761cf1/00000000-0000-0000-0000-00005f8f22d1"
 					(reference "Q3")
@@
 		(on_board yes)
 		(dnp no)
-		(property "Reference" "R11"
+		(property "Reference" "R17"
 			(at 133.35 67.31 90)
 			(effects
@@
 			)
 		)
-		(property "Footprint" "Resistor_SMD:R_0805_2012Metric_Pad1.15x1.40mm_HandSolder"
+		(property "Footprint" "Resistor_SMD:R_0805_2012Metric_Pad1.20x1.40mm_HandSolder"
 			(at 133.35 68.072 90)
 			(effects
@@
 		(instances
 			(project ""
-				(path "/dc0b64a3-156e-446d-a433-c56b0c761cf1/00000000-0000-0000-0000-00005f7bc591"
-					(reference "R11")
-					(unit 1)
-				)
 				(path "/dc0b64a3-156e-446d-a433-c56b0c761cf1/00000000-0000-0000-0000-00005f8f22d1"
 					(reference "R17")
@@
 		(on_board yes)
 		(dnp no)
-		(property "Reference" "R10"
+		(property "Reference" "R16"
 			(at 119.38 77.47 90)
 			(effects
@@
 			)
 		)
-		(property "Footprint" "Resistor_SMD:R_2512_6332Metric_Pad1.52x3.35mm_HandSolder"
+		(property "Footprint" "Resistor_SMD:R_2512_6332Metric_Pad1.40x3.35mm_HandSolder"
 			(at 123.698 78.74 90)
 			(effects
@@
 		(instances
 			(project ""
-				(path "/dc0b64a3-156e-446d-a433-c56b0c761cf1/00000000-0000-0000-0000-00005f7bc591"
-					(reference "R10")
-					(unit 1)
-				)
 				(path "/dc0b64a3-156e-446d-a433-c56b0c761cf1/00000000-0000-0000-0000-00005f8f22d1"
 					(reference "R16")
@@
 		(on_board yes)
 		(dnp no)
-		(property "Reference" "R14"
+		(property "Reference" "R18"
 			(at 134.62 54.61 90)
 			(effects
@@
 			)
 		)
-		(property "Footprint" "Resistor_SMD:R_0805_2012Metric_Pad1.15x1.40mm_HandSolder"
+		(property "Footprint" "Resistor_SMD:R_0805_2012Metric_Pad1.20x1.40mm_HandSolder"
 			(at 134.62 55.372 90)
 			(effects
@@
 		(instances
 			(project ""
-				(path "/dc0b64a3-156e-446d-a433-c56b0c761cf1/00000000-0000-0000-0000-00005f7bc591"
-					(reference "R14")
-					(unit 1)
-				)
 				(path "/dc0b64a3-156e-446d-a433-c56b0c761cf1/00000000-0000-0000-0000-00005f8f22d1"
 					(reference "R18")
@@
 		(on_board yes)
 		(dnp no)
-		(property "Reference" "C4"
+		(property "Reference" "C5"
 			(at 159.131 68.6816 0)
 			(effects
@@
 			)
 		)
-		(property "Footprint" "Capacitor_SMD:C_0805_2012Metric_Pad1.15x1.40mm_HandSolder"
+		(property "Footprint" "Capacitor_SMD:C_0805_2012Metric_Pad1.18x1.45mm_HandSolder"
 			(at 157.1752 73.66 0)
 			(effects
@@
 		(instances
 			(project ""
-				(path "/dc0b64a3-156e-446d-a433-c56b0c761cf1/00000000-0000-0000-0000-00005f7bc591"
-					(reference "C4")
-					(unit 1)
-				)
 				(path "/dc0b64a3-156e-446d-a433-c56b0c761cf1/00000000-0000-0000-0000-00005f8f22d1"
 					(reference "C5")
@@
 		(on_board yes)
 		(dnp no)
-		(property "Reference" "D2"
+		(property "Reference" "D3"
 			(at 111.76 78.74 90)
 			(effects
@@
 		(instances
 			(project ""
-				(path "/dc0b64a3-156e-446d-a433-c56b0c761cf1/00000000-0000-0000-0000-00005f7bc591"
-					(reference "D2")
-					(unit 1)
-				)
 				(path "/dc0b64a3-156e-446d-a433-c56b0c761cf1/00000000-0000-0000-0000-00005f8f22d1"
 					(reference "D3")
@@
 		(on_board yes)
 		(dnp no)
-		(property "Reference" "R9"
+		(property "Reference" "R15"
 			(at 113.03 73.66 90)
 			(effects
@@
 			)
 		)
-		(property "Footprint" "Resistor_SMD:R_0805_2012Metric_Pad1.15x1.40mm_HandSolder"
+		(property "Footprint" "Resistor_SMD:R_0805_2012Metric_Pad1.20x1.40mm_HandSolder"
 			(at 116.84 74.93 0)
 			(effects
@@
 		(instances
 			(project ""
-				(path "/dc0b64a3-156e-446d-a433-c56b0c761cf1/00000000-0000-0000-0000-00005f7bc591"
-					(reference "R9")
-					(unit 1)
-				)
 				(path "/dc0b64a3-156e-446d-a433-c56b0c761cf1/00000000-0000-0000-0000-00005f8f22d1"
 					(reference "R15")
