File: BMS/BMS.kicad_sch (KiCad schematic)
At the start: 43 parts, among them J1 Cell Taps, J2 Temp Sensors, J3 IsoSPI, J4 IsoSPI, Q1 NSV1C201MZ4, SW1 SW_DIP_x04, U1 LTC6811, U2 ADG708

Commit message: BMS Schema Done!
hello world
Parts:
- removed F1: Polyfuse, Fuse:Fuse_1812_4532Metric_Pad1.30x3.40mm_HandSolder, symbol Device:Polyfuse
- removed J1: Cell Taps, Connector_Molex:Molex_Nano-Fit_105313-xx08_1x08_P2.50mm_Horizontal, symbol Connector:Conn_01x08_Pin
- removed J2: Temp Sensors, Connector_Molex:Molex_Nano-Fit_105314-xx14_2x07_P2.50mm_Horizontal, symbol Connector_Generic:Conn_02x07_Top_Bottom
- removed SW1: SW_DIP_x04, FSFootprints:DIP A6H-4101, symbol Switch:SW_DIP_x04
- removed U1: LTC6811, 1FS_2_Global_Footprint_Library:FSOP-48_[LTC6811-2], symbol FSSymbols:LTC6811
- added 6_2_Pin_Connectors1, 6_2_Pin_Connectors2, 6_2_Pin_Connectors3, 6_2_Pin_Connectors4, 6_2_Pin_Connectors5, 6_2_Pin_Connectors6: ~, Connector_Molex:Molex_Nano-Fit_105313-xx02_1x02_P2.50mm_Horizontal, symbol Connector_Generic:Conn_02x01
- added H1, H2, H3, H4, H5: MountingHole_Pad, MountingHole:MountingHole_3.2mm_M3_DIN965_Pad, symbol Mechanical:MountingHole_Pad
- added J1: Conn_01x02_Pin, Connector_Molex:Molex_Nano-Fit_105313-xx02_1x02_P2.50mm_Horizontal, symbol Connector:Conn_01x02_Pin
- added R4: 10k, Resistor_SMD:R_0805_2012Metric_Pad1.20x1.40mm_HandSolder, symbol Device:R
- added SW2: A6H-4101, FS_3_Global_Footprint_Library:SW_A6H-4101_OMR, symbol FS_3_Global_Symbol_Library:A6H-4101
- added U3: LTC6811IG-2-TRPBF, FS_3_Global_Footprint_Library:LTC6811-2, symbol FS_3_Global_Symbol_Library:LTC6811IG-2-TRPBF
- C1, C12, C13, C2, C3, C6, C7, R3: footprint Capacitor_SMD:C_0805_2012Metric_Pad1.15x1.40mm_HandSolder -> Capacitor_SMD:C_0805_2012Metric_Pad1.18x1.45mm_HandSolder
- L1: footprint FSFootprints:HM2113ZNL -> FS_3_Global_Footprint_Library:HM2113ZNLT
- R1, R12, R13, R2, R32, R33, R37, R38, R39, R40, R41, R5, R51, R6, R7, R8: footprint Resistor_SMD:R_0805_2012Metric_Pad1.15x1.40mm_HandSolder -> Resistor_SMD:R_0805_2012Metric_Pad1.20x1.40mm_HandSolder
Connections:
- net BB6/B#+1 is gone; now on net BB5/B#+1: R1.2, R2.2
- net A0: now also SW2.4, U3.45 (A0)
- net A1: now also SW2.3, U3.46 (A1)
- net C0: now also U3.26 (C0)
- net C1: now also U3.24 (C1)
- net C2: now also U3.22 (C2)
- net C3: now also U3.14 (C6), U3.16 (C5), U3.18 (C4), U3.20 (C3)
- net C7: now also U3.12 (C7)
- net C8: now also U3.10 (C8)
- net C9-12: now also U3.2 (C12), U3.4 (C11), U3.6 (C10), U3.8 (C9)
- net DRV: now also U3.38 (DRIVE)
- net IBIAS: now also U3.44 (SDO(IBIAS))
- net ICMP: now also U3.43 (SDI(IMCP))
- net IsoSPI_N: now also U3.41 (CSB(IMA))
- net IsoSPI_P: now also SW2.1, U3.42 (SCK(IPA))
- net MUX_A0: now also U3.27 (GPIO1)
- net MUX_A1: now also U3.28 (GPIO2)
- net MUX_A2: now also U3.29 (GPIO3)
- net S1: now also U3.25 (S1)
- net S2: now also U3.23 (S2)
- net S3: now also U3.21 (S3)
- net S7: now also U3.13 (S7)
- net S8: now also U3.11 (S8)
- net S9: now also U3.9 (S9)
- net TEMP: now also U3.32 (GPIO4)
- net V+: now also U3.1 (V+)
- net V-: now also 6_2_Pin_Connectors1.1 (Pin_1), 6_2_Pin_Connectors2.1 (Pin_1), 6_2_Pin_Connectors3.1 (Pin_1), 6_2_Pin_Connectors4.1 (Pin_1), 6_2_Pin_Connectors5.1 (Pin_1), 6_2_Pin_Connectors6.1 (Pin_1), R4.2, U3.30 (V-), U3.31 (V-), U3.36 (DTEN), U3.48 (A3)
- net VREG: now also SW2.5, SW2.6, SW2.7, U3.37 (VREG), U3.40 (ISOMD)
- net at D9.1 (K): now also U3.33 (GPIO5)
- net at C6.2: now also U3.34 (VREF2)
- net at C7.2: now also U3.35 (VREF1)
- net at F8.2: now also J1.2 (Pin_2)
- net at F7.2: now also H1.1
- net at F6.2: now also H2.1
- net at F5.2: now also H3.1
- net at F4.2: now also H4.1
- net at F3.2: now also H5.1
- net at F2.2: now also J1.1 (Pin_1)
- net at R5.2: now also SW2.8
- net at U2.11 (S6): now also 6_2_Pin_Connectors6.2 (Pin_2)
- net at U2.12 (S5): now also 6_2_Pin_Connectors5.2 (Pin_2)
- net at U2.4 (S1): now also 6_2_Pin_Connectors1.2 (Pin_2)
- net at U2.5 (S2): now also 6_2_Pin_Connectors2.2 (Pin_2)
- net at U2.6 (S3): now also 6_2_Pin_Connectors3.2 (Pin_2)
- net at U2.7 (S4): now also 6_2_Pin_Connectors4.2 (Pin_2)
- new net A2: R4.1, SW2.2, U3.47 (A2)
- no-connect marks 8 -> 10
Other:
- removed sheet BB6
- note added: "1: ISOSpi Termintion 2: Address bit 2 3: Address bit 1 4: Address bit 0"
- note removed: "1: LTC6811 Power 2: ISOSpi Termintion 3: Address bit 1 4: Address bit 0"
- note removed: "B0"
- moved on the sheet: C1, C12, C13, C2, C3, C6, C7, D1, D9, J3, J4, L1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

Commit message: Fixed temp sense connector reference designators
Parts:
- renumbered J4 to J2, 6_2_Pin_Connectors1 to J4, 6_2_Pin_Connectors2 to J5, 6_2_Pin_Connectors3 to J6, 6_2_Pin_Connectors4 to J7, 6_2_Pin_Connectors5 to J8, 6_2_Pin_Connectors6 to J9
Changed lines of the file:
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@@
 		(on_board yes)
 		(dnp no)
-		(property "Reference" "J4"
+		(property "Reference" "J2"
 			(at 343.5858 115.062 0)
 			(effects
@@
 			(project ""
 				(path "/dc0b64a3-156e-446d-a433-c56b0c761cf1"
-					(reference "J4")
+					(reference "J2")
 					(unit 1)
 				)
@@
 		(on_board yes)
 		(dnp no)
-		(property "Reference" "6_2_Pin_Connectors6"
-			(at 298.196 181.102 0)
+		(property "Reference" "J9"
+			(at 299.466 185.42 0)
 			(effects
 				(font
@@
 			(project "BMS"
 				(path "/dc0b64a3-156e-446d-a433-c56b0c761cf1"
-					(reference "6_2_Pin_Connectors6")
+					(reference "J9")
 					(unit 1)
 				)
@@
 		(on_board yes)
 		(dnp no)
-		(property "Reference" "6_2_Pin_Connectors4"
-			(at 298.196 176.022 0)
+		(property "Reference" "J7"
+			(at 299.466 180.34 0)
 			(effects
 				(font
@@
 			(project "BMS"
 				(path "/dc0b64a3-156e-446d-a433-c56b0c761cf1"
-					(reference "6_2_Pin_Connectors4")
+					(reference "J7")
 					(unit 1)
 				)
@@
 		(on_board yes)
 		(dnp no)
-		(property "Reference" "6_2_Pin_Connectors2"
-			(at 298.196 170.942 0)
+		(property "Reference" "J5"
+			(at 299.466 175.26 0)
 			(effects
 				(font
@@
 			(project "BMS"
 				(path "/dc0b64a3-156e-446d-a433-c56b0c761cf1"
-					(reference "6_2_Pin_Connectors2")
+					(reference "J5")
 					(unit 1)
 				)
@@
 		(on_board yes)
 		(dnp no)
-		(property "Reference" "6_2_Pin_Connectors1"
-			(at 298.196 168.402 0)
+		(property "Reference" "J4"
+			(at 299.466 172.72 0)
 			(effects
 				(font
@@
 			(project "BMS"
 				(path "/dc0b64a3-156e-446d-a433-c56b0c761cf1"
-					(reference "6_2_Pin_Connectors1")
+					(reference "J4")
 					(unit 1)
 				)
@@
 		(on_board yes)
 		(dnp no)
-		(property "Reference" "6_2_Pin_Connectors3"
-			(at 298.196 173.482 0)
+		(property "Reference" "J6"
+			(at 299.466 177.8 0)
 			(effects
 				(font
@@
 			(project "BMS"
 				(path "/dc0b64a3-156e-446d-a433-c56b0c761cf1"
-					(reference "6_2_Pin_Connectors3")
+					(reference "J6")
 					(unit 1)
 				)
@@
 		(on_board yes)
 		(dnp no)
-		(property "Reference" "6_2_Pin_Connectors5"
-			(at 298.196 178.562 0)
+		(property "Reference" "J8"
+			(at 299.466 182.88 0)
 			(effects
 				(font
@@
 			(project "BMS"
 				(path "/dc0b64a3-156e-446d-a433-c56b0c761cf1"
-					(reference "6_2_Pin_Connectors5")
-					(unit 1)
-				)
+					(reference "J8")
+					(unit 1)
+				)

Commit message: Correct Fuse annotations
Parts:
- renumbered F8 to F1, F7 to F2, F6 to F3, F5 to F4, F4 to F5, F3 to F6, F2 to F7
Changed lines of the file:
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@@
 	(text "B6\n"
 		(exclude_from_sim no)
-		(at 72.644 70.104 0)
+		(at 74.168 69.85 0)
 		(effects
 			(font
@@
 	(text "B5\n"
 		(exclude_from_sim no)
-		(at 72.39 73.66 0)
+		(at 74.168 73.66 0)
 		(effects
 			(font
@@
 	(text "B4"
 		(exclude_from_sim no)
-		(at 72.39 77.47 0)
+		(at 74.168 77.47 0)
 		(effects
 			(font
@@
 	(text "B2\n"
 		(exclude_from_sim no)
-		(at 72.39 85.09 0)
+		(at 74.168 85.09 0)
 		(effects
 			(font
@@
 	(text "B7"
 		(exclude_from_sim no)
-		(at 72.898 66.294 0)
+		(at 74.168 66.04 0)
 		(effects
 			(font
@@
 	(text "B3\n"
 		(exclude_from_sim no)
-		(at 72.898 81.026 0)
+		(at 74.168 81.28 0)
 		(effects
 			(font
@@
 	(text "B1\n"
 		(exclude_from_sim no)
-		(at 73.152 88.646 0)
+		(at 74.168 88.646 0)
 		(effects
 			(font
@@
 		(on_board yes)
 		(dnp no)
-		(property "Reference" "F2"
-			(at 80.01 60.325 90)
+		(property "Reference" "F7"
+			(at 83.82 67.31 90)
 			(effects
 				(font
 					(size 1.27 1.27)
 				)
-				(hide yes)
 			)
 		)
@@
 			(project ""
 				(path "/dc0b64a3-156e-446d-a433-c56b0c761cf1"
-					(reference "F2")
+					(reference "F7")
 					(unit 1)
 				)
@@
 		(on_board yes)
 		(dnp no)
-		(property "Reference" "F3"
-			(at 80.01 64.135 90)
+		(property "Reference" "F6"
+			(at 83.82 71.12 90)
 			(effects
 				(font
 					(size 1.27 1.27)
 				)
-				(hide yes)
 			)
 		)
@@
 			(project ""
 				(path "/dc0b64a3-156e-446d-a433-c56b0c761cf1"
-					(reference "F3")
+					(reference "F6")
 					(unit 1)
 				)
@@
 		(on_board yes)
 		(dnp no)
-		(property "Reference" "F4"
-			(at 80.01 67.945 90)
+		(property "Reference" "F5"
+			(at 83.82 74.93 90)
 			(effects
 				(font
 					(size 1.27 1.27)
 				)
-				(hide yes)
 			)
 		)
@@
 			(project ""
 				(path "/dc0b64a3-156e-446d-a433-c56b0c761cf1"
-					(reference "F4")
+					(reference "F5")
 					(unit 1)
 				)
@@
 		(on_board yes)
 		(dnp no)
-		(property "Reference" "F5"
-			(at 80.01 71.755 90)
+		(property "Reference" "F4"
+			(at 83.82 78.74 90)
 			(effects
 				(font
 					(size 1.27 1.27)
 				)
-				(hide yes)
 			)
 		)
@@
 			(project ""
 				(path "/dc0b64a3-156e-446d-a433-c56b0c761cf1"
-					(reference "F5")
+					(reference "F4")
 					(unit 1)
 				)
@@
 		(on_board yes)
 		(dnp no)
-		(property "Reference" "F6"
-			(at 80.01 77.9018 90)
+		(property "Reference" "F3"
+			(at 83.82 82.55 90)
 			(effects
 				(font
 					(size 1.27 1.27)
 				)
-				(hide yes)
 			)
 		)
@@
 			(project ""
 				(path "/dc0b64a3-156e-446d-a433-c56b0c761cf1"
-					(reference "F6")
+					(reference "F3")
 					(unit 1)
 				)
@@
 		(on_board yes)
 		(dnp no)
-		(property "Reference" "F7"
-			(at 80.01 81.7118 90)
+		(property "Reference" "F2"
+			(at 83.82 86.36 90)
 			(effects
 				(font
 					(size 1.27 1.27)
 				)
-				(hide yes)
 			)
 		)
@@
 			(project ""
 				(path "/dc0b64a3-156e-446d-a433-c56b0c761cf1"
-					(reference "F7")
+					(reference "F2")
 					(unit 1)
 				)
@@
 		(on_board yes)
 		(dnp no)
-		(property "Reference" "F8"
-			(at 80.01 83.185 90)
+		(property "Reference" "F1"
+			(at 83.82 90.17 90)
 			(effects
 				(font
 					(size 1.27 1.27)
 				)
-				(hide yes)
 			)
 		)
@@
 			(project ""
 				(path "/dc0b64a3-156e-446d-a433-c56b0c761cf1"
-					(reference "F8")
+					(reference "F1")
 					(unit 1)
 				)

Commit message: Changed bms temp sense connectors to JST XH
Parts:
- J4, J5, J6, J7, J8, J9: footprint Connector_Molex:Molex_Nano-Fit_105313-xx02_1x02_P2.50mm_Horizontal -> Connector_JST:JST_XH_S2B-XH-A_1x02_P2.50mm_Horizontal
Changed lines of the file:
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@@
 			)
 		)
-		(property "Footprint" "Connector_Molex:Molex_Nano-Fit_105313-xx02_1x02_P2.50mm_Horizontal"
+		(property "Footprint" "Connector_JST:JST_XH_S2B-XH-A_1x02_P2.50mm_Horizontal"
 			(at 298.45 185.42 0)
 			(effects
@@
 			)
 		)
-		(property "Footprint" "Connector_Molex:Molex_Nano-Fit_105313-xx02_1x02_P2.50mm_Horizontal"
+		(property "Footprint" "Connector_JST:JST_XH_S2B-XH-A_1x02_P2.50mm_Horizontal"
 			(at 298.45 180.34 0)
 			(effects
@@
 			)
 		)
-		(property "Footprint" "Connector_Molex:Molex_Nano-Fit_105313-xx02_1x02_P2.50mm_Horizontal"
+		(property "Footprint" "Connector_JST:JST_XH_S2B-XH-A_1x02_P2.50mm_Horizontal"
 			(at 298.45 175.26 0)
 			(effects
@@
 			)
 		)
-		(property "Footprint" "Connector_Molex:Molex_Nano-Fit_105313-xx02_1x02_P2.50mm_Horizontal"
+		(property "Footprint" "Connector_JST:JST_XH_S2B-XH-A_1x02_P2.50mm_Horizontal"
 			(at 298.45 172.72 0)
 			(effects
@@
 			)
 		)
-		(property "Footprint" "Connector_Molex:Molex_Nano-Fit_105313-xx02_1x02_P2.50mm_Horizontal"
+		(property "Footprint" "Connector_JST:JST_XH_S2B-XH-A_1x02_P2.50mm_Horizontal"
 			(at 298.45 177.8 0)
 			(effects
@@
 			)
 		)
-		(property "Footprint" "Connector_Molex:Molex_Nano-Fit_105313-xx02_1x02_P2.50mm_Horizontal"
+		(property "Footprint" "Connector_JST:JST_XH_S2B-XH-A_1x02_P2.50mm_Horizontal"
 			(at 298.45 182.88 0)
 			(effects
