File: BMS_Alternative_1/BMS.kicad_sch (KiCad schematic)
At the start: 53 parts, among them J1 Conn_01x02_Pin, J2 IsoSPI, J3 IsoSPI, Q1 NSV1C201MZ4, SW2 A6H-4101, U2 ADG708, U3 LTC6811IG-2-TRPBF

Commit message: Fixed footprints and 3d models for bms
Parts:
- J1, J2, J3, J4, J5, J6, J7, J8, J9: footprint Connector_Molex:Molex_Nano-Fit_105313-xx02_1x02_P2.50mm_Horizontal -> FS_3_Global_Footprint_Library:Molex_Nano-Fit_105313-xx02_1x02_P2.50mm_Horizontal
Changed lines of the file:
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@@
 			)
 		)
-		(property "Footprint" "Connector_Molex:Molex_Nano-Fit_105313-xx02_1x02_P2.50mm_Horizontal"
+		(property "Footprint" "FS_3_Global_Footprint_Library:Molex_Nano-Fit_105313-xx02_1x02_P2.50mm_Horizontal"
 			(at 342.9 113.03 0)
 			(effects
@@
 			)
 		)
-		(property "Footprint" "Connector_Molex:Molex_Nano-Fit_105313-xx02_1x02_P2.50mm_Horizontal"
+		(property "Footprint" "FS_3_Global_Footprint_Library:Molex_Nano-Fit_105313-xx02_1x02_P2.50mm_Horizontal"
 			(at 342.9 118.11 0)
 			(effects
@@
 			)
 		)
-		(property "Footprint" "Connector_Molex:Molex_Nano-Fit_105313-xx02_1x02_P2.50mm_Horizontal"
+		(property "Footprint" "FS_3_Global_Footprint_Library:Molex_Nano-Fit_105313-xx02_1x02_P2.50mm_Horizontal"
 			(at 298.45 185.42 0)
 			(effects
@@
 			)
 		)
-		(property "Footprint" "Connector_Molex:Molex_Nano-Fit_105313-xx02_1x02_P2.50mm_Horizontal"
+		(property "Footprint" "FS_3_Global_Footprint_Library:Molex_Nano-Fit_105313-xx02_1x02_P2.50mm_Horizontal"
 			(at 298.45 180.34 0)
 			(effects
@@
 			)
 		)
-		(property "Footprint" "Connector_Molex:Molex_Nano-Fit_105313-xx02_1x02_P2.50mm_Horizontal"
+		(property "Footprint" "FS_3_Global_Footprint_Library:Molex_Nano-Fit_105313-xx02_1x02_P2.50mm_Horizontal"
 			(at 298.45 175.26 0)
 			(effects
@@
 			)
 		)
-		(property "Footprint" "Connector_Molex:Molex_Nano-Fit_105313-xx02_1x02_P2.50mm_Horizontal"
+		(property "Footprint" "FS_3_Global_Footprint_Library:Molex_Nano-Fit_105313-xx02_1x02_P2.50mm_Horizontal"
 			(at 298.45 172.72 0)
 			(effects
@@
 			)
 		)
-		(property "Footprint" "Connector_Molex:Molex_Nano-Fit_105313-xx02_1x02_P2.50mm_Horizontal"
+		(property "Footprint" "FS_3_Global_Footprint_Library:Molex_Nano-Fit_105313-xx02_1x02_P2.50mm_Horizontal"
 			(at 298.45 177.8 0)
 			(effects
@@
 			)
 		)
-		(property "Footprint" "Connector_Molex:Molex_Nano-Fit_105313-xx02_1x02_P2.50mm_Horizontal"
+		(property "Footprint" "FS_3_Global_Footprint_Library:Molex_Nano-Fit_105313-xx02_1x02_P2.50mm_Horizontal"
 			(at 298.45 182.88 0)
 			(effects
@@
 			)
 		)
-		(property "Footprint" "Connector_Molex:Molex_Nano-Fit_105313-xx02_1x02_P2.50mm_Horizontal"
+		(property "Footprint" "FS_3_Global_Footprint_Library:Molex_Nano-Fit_105313-xx02_1x02_P2.50mm_Horizontal"
 			(at 48.26 74.93 0)
 			(effects

Commit message: Changed bms temp sense connectors to JST XH
Parts:
- J4, J5, J6, J7, J8, J9: footprint FS_3_Global_Footprint_Library:Molex_Nano-Fit_105313-xx02_1x02_P2.50mm_Horizontal -> Connector_JST:JST_XH_S2B-XH-A_1x02_P2.50mm_Horizontal
Changed lines of the file:
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@@
 			)
 		)
-		(property "Footprint" "FS_3_Global_Footprint_Library:Molex_Nano-Fit_105313-xx02_1x02_P2.50mm_Horizontal"
+		(property "Footprint" "Connector_JST:JST_XH_S2B-XH-A_1x02_P2.50mm_Horizontal"
 			(at 298.45 185.42 0)
 			(effects
@@
 			)
 		)
-		(property "Footprint" "FS_3_Global_Footprint_Library:Molex_Nano-Fit_105313-xx02_1x02_P2.50mm_Horizontal"
+		(property "Footprint" "Connector_JST:JST_XH_S2B-XH-A_1x02_P2.50mm_Horizontal"
 			(at 298.45 180.34 0)
 			(effects
@@
 			)
 		)
-		(property "Footprint" "FS_3_Global_Footprint_Library:Molex_Nano-Fit_105313-xx02_1x02_P2.50mm_Horizontal"
+		(property "Footprint" "Connector_JST:JST_XH_S2B-XH-A_1x02_P2.50mm_Horizontal"
 			(at 298.45 175.26 0)
 			(effects
@@
 			)
 		)
-		(property "Footprint" "FS_3_Global_Footprint_Library:Molex_Nano-Fit_105313-xx02_1x02_P2.50mm_Horizontal"
+		(property "Footprint" "Connector_JST:JST_XH_S2B-XH-A_1x02_P2.50mm_Horizontal"
 			(at 298.45 172.72 0)
 			(effects
@@
 			)
 		)
-		(property "Footprint" "FS_3_Global_Footprint_Library:Molex_Nano-Fit_105313-xx02_1x02_P2.50mm_Horizontal"
+		(property "Footprint" "Connector_JST:JST_XH_S2B-XH-A_1x02_P2.50mm_Horizontal"
 			(at 298.45 177.8 0)
 			(effects
@@
 			)
 		)
-		(property "Footprint" "FS_3_Global_Footprint_Library:Molex_Nano-Fit_105313-xx02_1x02_P2.50mm_Horizontal"
+		(property "Footprint" "Connector_JST:JST_XH_S2B-XH-A_1x02_P2.50mm_Horizontal"
 			(at 298.45 182.88 0)
 			(effects
