File: Telemetry Main Board/Telemetry Board.kicad_sch (KiCad schematic)
At the start: 12 parts, among them J1 776180-1, U3 CD74HC4067SM96, U4 ISO1050DUB, U5 NUCLEO-L432KC

Commit message: Notes for new revision
Other:
- added sheet DEMO STUFF (untitled.kicad_sch)
- note added: "1 CAN bus -> 2 CAN Busses SPI Connected to 2 can controllers https://ww1.microchip.com/downloads/en/DeviceDoc/MCP2515-Stand-Alone-CAN-Controller-with-SPI-20001801J.pdf peripheral boards being replaced with CAN (Except power and ground) Make a list of sensors that need to be powered by PDB Reach out to AUTO companies for flow sensor(s) Update conneter to have power(and gnd), can x2, power to perip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"
Changed lines of the file:
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@@
 	(title_block
 		(title "Telemetry Board")
-		(date "2024-10-08")
+		(date "2024-10-24")
 		(rev "1.0")
 	)
@@
 	(text "Do Not Use\n"
 		(exclude_from_sim no)
+		(at 175.26 77.978 0)
+		(effects
+			(font
+				(size 1.27 1.27)
+			)
+			(justify left bottom)
+		)
+	)
+	(text "1 CAN bus -> 2 CAN Busses\nSPI Connected to 2 can controllers\nhttps://ww1.microchip.com/downloads/en/DeviceDoc/MCP2515-Stand-Alone-CAN-Controller-with-SPI-20001801J.pdf\nperipheral boards being replaced with CAN (Except power and ground)\nMake a list of sensors that need to be powered by PDB\nReach out to AUTO companies for flow sensor(s)\nUpdate conneter to have power(and gnd), can x2, power to peripherals (and gnd), direct inputs.\nDirect inputs go to multiplexer."
+		(exclude_from_sim no)
+		(at 149.352 -9.652 0)
+		(effects
+			(font
+				(size 1.27 1.27)
+			)
+		)
+	)
+	(text "Do Not Use\n"
+		(exclude_from_sim no)
 		(at 175.26 52.07 0)
 		(effects
@@
 				)
 			)
+		)
+	)
+	(sheet
+		(at 226.06 30.48)
+		(size 39.37 26.67)
+		(fields_autoplaced yes)
+		(stroke
+			(width 0.1524)
+			(type solid)
+		)
+		(fill
+			(color 0 0 0 0.0000)
+		)
+		(property "Sheetname" "DEMO STUFF"
+			(at 226.06 29.7684 0)
+			(effects
+				(font
+					(size 1.27 1.27)
+				)
+				(justify left bottom)
+			)
+		)
+		(property "Sheetfile" "untitled.kicad_sch"
+			(at 226.06 57.7346 0)
+			(effects
+				(font
+					(size 1.27 1.27)
+				)
+				(justify left top)
+			)
+		)
+		(instances
+			(project "Telemetry Board"
+				(path "/dde73ecd-f7ea-407a-a1ab-cf1927044ecb"
+					(page "3")
+				)
+			)
