File: Telemetry Main Board/Telemetry Main Board.kicad_sch (KiCad schematic)
At the start: 12 parts, among them J1 776180-1, U3 CD74HC4067SM96, U4 ISO1050DUB, U5 NUCLEO-L432KC

Commit message: Telemetry board update
replaces old telemetry board with the new updated one
Parts:
- added C10, C11, C12, C6: 100nf, Capacitor_SMD:C_0805_2012Metric_Pad1.18x1.45mm_HandSolder, symbol Device:C
- added U7, U9: MCP2515-I/SO, Package_SO:SOIC-18W_7.5x11.6mm_P1.27mm, symbol FS_3_Global_Symbol_Library:MCP2515-I_SO
- added U8: ISO1050DUB, Package_SO:SOP-8_6.62x9.15mm_P2.54mm, symbol Interface_CAN_LIN:ISO1050DUB
Connections:
- net +12V: now also J1.2; no longer J1.14
- net +3V3: now also J1.12, C10.2, U8.1 (VCC1); no longer J1.20, J1.26, J1.3, J1.32, J1.9
- net +5V: now also C6.2, U8.8 (VCC2); no longer J1.2, J1.25, J1.31, J1.8
- net Brake Sensor B: now also J1.15; no longer J1.23
- net Brake Sensor F: now also J1.14; no longer J1.22
- net GND: now also J1.11, C10.1, C11.2, C12.2, C6.1, U7.9 (VSS), U8.4 (GND1), U8.5 (GND2), U9.9 (VSS); no longer J1.13, J1.19, J1.24, J1.30, J1.7
- net Steering Sensor: now also J1.13; no longer J1.21
- net SPI3_SSEL1: now reaches U5.CN3_1 (PA9)
- net SPI3_SSEL1: now also U9.16 (*CS)
- net SPI3-MOSI: now reaches U5.CN3_14 (PB5)
- net SPI3-MISO: now reaches U5.CN3_15 (PB4)
- net SPI3_SSEL2: now reaches U5.CN3_2 (PA10)
- net SPI3_SSEL2: now also U7.16 (*CS)
- net SPI3-SCLK: now reaches U5.CN4_15 (PB3)
- net CAN1_RD: no longer names the net of U5.CN3_13 (PA11)
- net CAN1_RD: no longer U4.2 (RXD)
- net CAN1_TD: no longer names the net of U5.CN3_5 (PA12)
- net CAN1_TD: no longer U4.3 (TXD)
- removed net CAN_H: J1.15, J1.17, U4.7 (CANH)
- removed net CAN_L: J1.16, J1.18, U4.6 (CANL)
- net Shock Position BL: no longer names the net of U3.19 (I12)
- net Shock Position BL: no longer J1.33
- net Shock Position BR: no longer names the net of U3.22 (I9)
- net Shock Position BR: no longer J1.27
- net Shock Position FL renamed Acc Intake Flow Rate
- net Acc Intake Flow Rate: now also J1.19; no longer J1.10
- net Shock Position FR renamed Acc Intake Temp
- net Acc Intake Temp: now also J1.16; no longer J1.4
- net Strain BL: no longer names the net of U3.18 (I13)
- net Strain BL: no longer J1.34
- net Strain BR: no longer names the net of U3.21 (I10)
- net Strain BR: no longer J1.28
- net Strain FL: no longer names the net of U3.2 (I7)
- net Strain FL: no longer J1.11
- net Strain FR renamed Acc Exhaust Temp
- net Acc Exhaust Temp: now also J1.17; no longer J1.5
- net Wheel Speed BL: no longer names the net of U3.17 (I14)
- net Wheel Speed BL: no longer J1.35
- net Wheel Speed BR: no longer names the net of U3.20 (I11)
- net Wheel Speed BR: no longer J1.29
- net Wheel Speed FL: no longer names the net of U3.23 (I8)
- net Wheel Speed FL: no longer J1.12
- net Wheel Speed FR renamed Acc Intake Pressure
- net Acc Intake Pressure: now also J1.18; no longer J1.6
- new net +3.3V: C11.1, C12.1, U7.18 (VDD), U9.18 (VDD)
- new net CAN1_H: J1.3, J1.4, U4.7 (CANH)
- new net CAN1_L: J1.7, J1.8, U4.6 (CANL)
- new net CAN1_RX: U4.2 (RXD), U9.2 (RXCAN)
- new net CAN1_TX: U4.3 (TXD), U9.1 (TXCAN)
- new net CAN2_H: J1.5, J1.6, U8.7 (CANH)
- new net CAN2_L: J1.10, J1.9, U8.6 (CANL)
- new net CAN2_RX: U7.2 (RXCAN), U8.2 (RXD)
- new net CAN2_TX: U7.1 (TXCAN), U8.3 (TXD)
- new net SPI3_MISO: U7.15 (SO), U9.15 (SO)
- new net SPI3_MOSI: U7.14 (SI), U9.14 (SI)
- new net SPI3_SCLK: U7.13 (SCK), U9.13 (SCK)
- no-connect marks 21 -> 18
Other:
- removed sheet DEMO STUFF
- note added: "1 CAN bus -> 2 CAN Busses SPI Connected to 2 can controllers https://ww1.microchip.com/downloads/en/DeviceDoc/MCP2515-Stand-Alone-CAN-Controller-with-SPI-20001801J.pdf peripheral boards being replaced with CAN (Except power and ground) Make a list of sensors that need to be powered by PDB Reach out to AUTO companies for flow sensor(s) Update connector to have power(and gnd), can x2, power to peri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"
- note added: "35 pin connector"
- note added: "CAN to SPI"
- note added: "CAN1 transceiver"
- note added: "CAN2 transceiver"
- note added: "Microcontroller"
- note added: "Multiplexer"
- note removed: "1 CAN bus -> 2 CAN Busses SPI Connected to 2 can controllers https://ww1.microchip.com/downloads/en/DeviceDoc/MCP2515-Stand-Alone-CAN-Controller-with-SPI-20001801J.pdf peripheral boards being replaced with CAN (Except power and ground) Make a list of sensors that need to be powered by PDB Reach out to AUTO companies for flow sensor(s) Update conneter to have power(and gnd), can x2, power to perip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"
- note removed: "CAN transciever"
- moved on the sheet: C7, C8, C9, U4, U5A
