File: ETC/ETC.kicad_sch (KiCad schematic)
At the start: 30 parts, among them P1 DTM1312PC12PDR008, U1 NUCLEO-F446RE, U2 MCP6004, U3 LM7805_TO220, U4 LM7809_TO220, U5 ISO1050DUB, U6 ISO1050DUB, U7 SN74AHC14N

Commit message: ETC Schematic Rev. 1
Parts:
- removed unit 3 of U1
- added C10, C11, C12, C13: 100nF, Capacitor_SMD:C_0805_2012Metric_Pad1.18x1.45mm_HandSolder, symbol Device:C
- added R14, R15: 120Ω, Resistor_SMD:R_0805_2012Metric_Pad1.20x1.40mm_HandSolder, symbol Device:R
- added unit 4 of U2
- C1, C2, C3, C4: footprint (none) -> Capacitor_SMD:C_0805_2012Metric_Pad1.18x1.45mm_HandSolder
- C8, C9: value 10 nF -> 100 nF; footprint (none) -> Capacitor_SMD:C_0805_2012Metric_Pad1.18x1.45mm_HandSolder
- P1: footprint TE_DTM1312PC12PDR008 -> FS_3_Global_Footprint_Library:TE_DTM1312PC12PDR008
- R10, R12: value 180kΩ -> 10kΩ
- R11, R13: value 10kΩ -> 390kΩ; footprint (none) -> Resistor_SMD:R_0805_2012Metric_Pad1.20x1.40mm_HandSolder
- U1: footprint NUCLEO-F446RE:MODULE_NUCLEO-F446RE -> FS_3_Global_Footprint_Library:NUCLEO-F446RE
- U2: footprint (none) -> FS_3_Global_Footprint_Library:N14
- U7: footprint N14 -> FS_3_Global_Footprint_Library:N14
Connections:
- net +3V3: now also U1.CN7_16 (CN7_+3V3), U5.1 (VCC1), U6.1 (VCC1), C10.1, C12.1
- net +5V: now also U5.8 (VCC2), U6.8 (VCC2), C11.1, C13.1
- net +9V: now also U1.CN7_24 (CN7_VIN)
- net BSE: now also U1.CN7_38 (PC0/PB8)
- net Cockpit_Signal: now also U1.CN7_31 (PH1)
- net GND: now also U1.CN10_20 (CN10_GND__1), U1.CN10_32 (AGND), U1.CN10_9 (CN10_GND), U1.CN7_19 (CN7_GND__1), U1.CN7_20 (CN7_GND__2), U1.CN7_22 (CN7_GND__3), U1.CN7_8 (CN7_GND), U5.4 (GND1), U5.5 (GND2), U6.4 (GND1), U6.5 (GND2), U7.10 (5Y), U7.11 (5A), U7.12 (6Y), U7.13 (6A), U7.5 (3A), U7.6 (3Y), U7.8 (4Y), U7.9 (4A), C10.2, C11.2, C12.2, C13.2
- net HE1: now also U1.CN7_28 (PA0)
- net HE2: now also U1.CN7_34 (PB0)
- net H_CAN: now also U6.7 (CANH), R15.1
- net H_Motor_CAN: now also U5.7 (CANH), R14.1
- net L_CAN: now also U6.6 (CANL), R15.2
- net L_Motor_CAN: now also U5.6 (CANL), R14.2
- net RTDS: now also U1.CN7_23 (PC13)
- net Reverse_Signal: now also U1.CN7_27 (PC15)
- net CAN_RD: now reaches U6.2 (RXD)
- net CAN_RD: now also U1.CN10_29 (PB5)
- net CAN_TD: now reaches U6.3 (TXD)
- net CAN_TD: now also U1.CN10_17 (PB6)
- net Motor_CAN_TD: now reaches U1.CN10_12 (PA12)
- net Motor_CAN_TD: now also U5.3 (TXD)
- net Motor_CAN_RD: now reaches U1.CN10_14 (PA11)
- net Motor_CAN_RD: now also U5.2 (RXD)
- no-connect marks 0 -> 56
Other:
- note added: "9V and 5V Linear Regulators"
- note added: "Analog Input Scaling"
- note added: "CAN Trancievers"
- note added: "DTM Connector"
- note added: "Digital Input Debouncing"
- note added: "Inverting Schmitt Trigger"
- note added: "MCU Connections"
- company: (none) -> Dustin Wang - Formula Slug
- title: (none) -> ETC
- moved on the sheet: C1, C2, C3, C4, C5, C6, C7, C8, C9, P1, R1, R10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

Commit message: Rev. 1.1: floating pins R bad
Connections:
- net GND: now also U2.12 (+); no longer U7.10 (5Y), U7.12 (6Y), U7.6 (3Y), U7.8 (4Y)
- net at U2.13 (-): now also U2.14
- no-connect marks 56 -> 57

Commit message: NUCLEO F446RE footprint fix
Other:
- moved on the sheet: R10, R11
Changed lines of the file:
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@@
 	(wire
 		(pts
-			(xy 44.45 223.52) (xy 53.34 223.52)
+			(xy 44.45 223.52) (xy 50.8 223.52)
 		)
 		(stroke
@@
 	(wire
 		(pts
-			(xy 44.45 213.36) (xy 44.45 214.63)
+			(xy 44.45 208.28) (xy 44.45 209.55)
+		)
+		(stroke
+			(width 0)
+			(type default)
+		)
+	)
+	(wire
+		(pts
+			(xy 44.45 217.17) (xy 44.45 223.52)
 		)
 		(stroke
@@
 	(wire
 		(pts
-			(xy 44.45 222.25) (xy 44.45 223.52)
-		)
-		(stroke
-			(width 0)
-			(type default)
-		)
-	)
-	(wire
-		(pts
 			(xy 134.62 106.68) (xy 144.78 106.68)
 		)
@@
 	(wire
 		(pts
-			(xy 60.96 223.52) (xy 66.04 223.52)
+			(xy 58.42 223.52) (xy 66.04 223.52)
 		)
 		(stroke
@@
 	(symbol
 		(lib_id "power:+3V3")
-		(at 44.45 213.36 0)
+		(at 44.45 208.28 0)
 		(unit 1)
 		(exclude_from_sim no)
@@
 		(fields_autoplaced yes)
 		(property "Reference" "#PWR029"
-			(at 44.45 217.17 0)
+			(at 44.45 212.09 0)
 			(effects
 				(font
@@
 		)
 		(property "Value" "+3V3"
-			(at 44.45 208.28 0)
+			(at 44.45 203.2 0)
 			(effects
 				(font
@@
 		)
 		(property "Footprint" ""
-			(at 44.45 213.36 0)
+			(at 44.45 208.28 0)
 			(effects
 				(font
@@
 		)
 		(property "Datasheet" ""
-			(at 44.45 213.36 0)
+			(at 44.45 208.28 0)
 			(effects
 				(font
@@
 		)
 		(property "Description" "Power symbol creates a global label with name \"+3V3\""
-			(at 44.45 213.36 0)
+			(at 44.45 208.28 0)
 			(effects
 				(font
@@
 	(symbol
 		(lib_id "Device:R")
-		(at 44.45 218.44 0)
+		(at 44.45 213.36 0)
 		(unit 1)
 		(exclude_from_sim no)
@@
 		(fields_autoplaced yes)
 		(property "Reference" "R10"
-			(at 46.99 217.17 0)
+			(at 46.99 212.09 0)
 			(effects
 				(font
@@
 		)
 		(property "Value" "10kΩ"
-			(at 46.99 219.71 0)
+			(at 46.99 214.63 0)
 			(effects
 				(font
@@
 		)
 		(property "Footprint" "Resistor_SMD:R_0805_2012Metric_Pad1.20x1.40mm_HandSolder"
-			(at 42.672 218.44 90)
+			(at 42.672 213.36 90)
 			(effects
 				(font
@@
 		)
 		(property "Datasheet" "~"
-			(at 44.45 218.44 0)
+			(at 44.45 213.36 0)
 			(effects
 				(font
@@
 		)
 		(property "Description" ""
-			(at 44.45 218.44 0)
+			(at 44.45 213.36 0)
 			(effects
 				(font
@@
 	(symbol
 		(lib_id "Device:R")
-		(at 57.15 223.52 270)
+		(at 54.61 223.52 270)
 		(unit 1)
 		(exclude_from_sim no)
@@
 		(fields_autoplaced yes)
 		(property "Reference" "R11"
-			(at 57.15 217.17 90)
+			(at 54.61 217.17 90)
 			(effects
 				(font
@@
 		)
 		(property "Value" "390kΩ"
-			(at 57.15 219.71 90)
+			(at 54.61 219.71 90)
 			(effects
 				(font
@@
 		)
 		(property "Footprint" "Resistor_SMD:R_0805_2012Metric_Pad1.20x1.40mm_HandSolder"
-			(at 57.15 221.742 90)
+			(at 54.61 221.742 90)
 			(effects
 				(font
@@
 		)
 		(property "Datasheet" "~"
-			(at 57.15 223.52 0)
+			(at 54.61 223.52 0)
 			(effects
 				(font
@@
 		)
 		(property "Description" "Resistor"
-			(at 57.15 223.52 0)
+			(at 54.61 223.52 0)
 			(effects
 				(font

Commit message: Remove schmitt trigger
Parts:
- removed C8, C9: 100 nF, Capacitor_SMD:C_0805_2012Metric_Pad1.18x1.45mm_HandSolder, symbol Device:C
- removed R10, R12: 10kΩ, Resistor_SMD:R_0805_2012Metric_Pad1.20x1.40mm_HandSolder, symbol Device:R
- removed R11, R13: 390kΩ, Resistor_SMD:R_0805_2012Metric_Pad1.20x1.40mm_HandSolder, symbol Device:R
- removed U7: SN74AHC14N, FS_3_Global_Footprint_Library:N14, symbol FS_3_Global_Symbol_Library:SN74AHC14N
- added C14, C15: 100 nF, Capacitor_SMD:C_0805_2012Metric_Pad1.18x1.45mm_HandSolder, symbol Device:C
- added R16, R18: 1kΩ, Resistor_SMD:R_0805_2012Metric_Pad1.20x1.40mm_HandSolder, symbol Device:R
- added R17, R19: 200kΩ, Resistor_SMD:R_0805_2012Metric_Pad1.20x1.40mm_HandSolder, symbol Device:R
Connections:
- net +3V3: now also R16.1, R18.1
- net Cockpit_Raw: now also R16.2, R17.2
- net Cockpit_Signal: now also C14.1, R17.1
- net GND: now also C14.2, C15.2
- net Reverse_Raw: now also R18.2, R19.2
- net Reverse_Signal: now also C15.1, R19.1
- no-connect marks 57 -> 53
Other:
- note removed: "Inverting Schmitt Trigger"

Commit message: save work on brake light schematic update
Parts:
- added D1: LED, LED_SMD:LED_0805_2012Metric_Pad1.15x1.40mm_HandSolder, symbol Device:LED
Connections:
- net GND: now also P1.C4, D1.1 (K)
- net Brake_Power: now reaches P1.C3
- net Brake_Power: now also D1.2 (A)
- net Brake_Signal: now reaches U1.CN7_25 (PC14)
- no-connect marks 53 -> 50
Other:
- note added: "Brake"
- note added: "Brake Light and RTDS Switching"

Commit message: add transistor to brake light circuit
Parts:
- removed D1: LED, LED_SMD:LED_0805_2012Metric_Pad1.15x1.40mm_HandSolder, symbol Device:LED
- added U7: SSM6N37FU_LF, Package_TO_SOT_SMD:SOT-363_SC-70-6_Handsoldering, symbol FS_3_Global_Symbol_Library:SSM6N37FU_LF
Connections:
- net Brake_Power is gone; now on net GND: P1.C3
- net +12V: now also U7.1
- net Brake_Signal: now also U7.2
- net GND: now also U7.6
- no-connect marks 50 -> 53
Changed lines of the file:
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@@
 	)
 	(junction
-		(at 48.26 226.06)
+		(at 111.76 217.17)
 		(diameter 0)
 		(color 0 0 0 0)
@@
 	)
 	(no_connect
+		(at 45.72 251.46)
+	)
+	(no_connect
 		(at 321.31 110.49)
 	)
@@
 	)
 	(no_connect
+		(at 111.76 251.46)
+	)
+	(no_connect
 		(at 351.79 128.27)
 	)
@@
 	)
 	(no_connect
+		(at 111.76 234.95)
+	)
+	(no_connect
 		(at 351.79 168.91)
 	)
@@
 	(wire
 		(pts
-			(xy 48.26 234.95) (xy 48.26 236.22)
-		)
-		(stroke
-			(width 0)
-			(type default)
-		)
-	)
-	(wire
-		(pts
 			(xy 321.31 186.69) (xy 321.31 189.23)
 		)
@@
 	(wire
 		(pts
-			(xy 48.26 226.06) (xy 62.23 226.06)
+			(xy 111.76 217.17) (xy 125.73 217.17)
 		)
 		(stroke
@@
 	(wire
 		(pts
-			(xy 21.59 215.9) (xy 35.56 215.9)
+			(xy 31.75 245.11) (xy 45.72 245.11)
 		)
 		(stroke
@@
 	(wire
 		(pts
-			(xy 48.26 223.52) (xy 48.26 226.06)
+			(xy 111.76 214.63) (xy 111.76 217.17)
 		)
 		(stroke
@@
 	(wire
 		(pts
-			(xy 48.26 227.33) (xy 48.26 226.06)
+			(xy 111.76 217.17) (xy 111.76 219.71)
 		)
 		(stroke
@@
 	(rectangle
 		(start 17.78 189.23)
-		(end 120.65 250.19)
+		(end 138.43 278.13)
 		(stroke
 			(width 0)
@@
 	(text "Brake Light and RTDS Switching"
 		(exclude_from_sim no)
-		(at 68.326 245.11 0)
+		(at 77.47 272.796 0)
 		(effects
 			(font
@@
 	)
 	(label "Brake_Signal"
-		(at 21.59 215.9 0)
+		(at 31.75 245.11 0)
 		(fields_autoplaced yes)
 		(effects
@@
 	)
 	(label "Brake_Power"
-		(at 62.23 226.06 180)
+		(at 125.73 217.17 180)
 		(fields_autoplaced yes)
 		(effects
@@
 	)
 	(symbol
+		(lib_id "FS_3_Global_Symbol_Library:SSM6N37FU_LF")
+		(at 45.72 214.63 0)
+		(unit 1)
+		(exclude_from_sim no)
+		(in_bom yes)
+		(on_board yes)
+		(dnp no)
+		(fields_autoplaced yes)
+		(property "Reference" "U7"
+			(at 78.74 199.39 0)
+			(effects
+				(font
+					(size 1.524 1.524)
+				)
+			)
+		)
+		(property "Value" "SSM6N37FU_LF"
+			(at 78.74 201.93 0)
+			(effects
+				(font
+					(size 1.524 1.524)
+				)
+			)
+		)
+		(property "Footprint" "Package_TO_SOT_SMD:SOT-363_SC-70-6_Handsoldering"
+			(at 45.72 214.63 0)
+			(effects
+				(font
+					(size 1.27 1.27)
+					(italic yes)
+				)
+				(hide yes)
+			)
+		)
+		(property "Datasheet" "SSM6N37FU_LF"
+			(at 45.72 214.63 0)
+			(effects
+				(font
+					(size 1.27 1.27)
+					(italic yes)
+				)
+				(hide yes)
+			)
+		)
+		(property "Description" "High Speed NMOS"
+			(at 45.72 214.63 0)
+			(effects
+				(font
+					(size 1.27 1.27)
+				)
+				(hide yes)
+			)
+		)
+		(pin "2"
+		)
+		(pin "3"
+		)
+		(pin "4"
+		)
+		(pin "5"
+		)
+		(pin "6"
+		)
+		(pin "1"
+		)
+		(instances
+			(project ""
+				(path "/61e913ea-868b-4b77-8707-03788b798f2b"
+					(reference "U7")
+					(unit 1)
+				)
+			)
+		)
+	)
+	(symbol
 		(lib_id "Device:C")
 		(at 233.68 123.19 0)
@@
 	(symbol
 		(lib_id "power:+12V")
-		(at 48.26 205.74 0)
+		(at 45.72 214.63 90)
 		(unit 1)
 		(exclude_from_sim no)
@@
 		(dnp no)
 		(property "Reference" "#PWR030"
-			(at 48.26 209.55 0)
+			(at 49.53 214.63 0)
 			(effects
 				(font
@@
 		)
 		(property "Value" "+12V"
-			(at 48.2601 201.93 90)
+			(at 41.91 214.6299 90)
 			(effects
 				(font
@@
 		)
 		(property "Footprint" ""
-			(at 48.26 205.74 0)
+			(at 45.72 214.63 0)
 			(effects
 				(font
@@
 		)
 		(property "Datasheet" ""
-			(at 48.26 205.74 0)
+			(at 45.72 214.63 0)
 			(effects
 				(font
@@
 		)
 		(property "Description" "Power symbol creates a global label with name \"+12V\""
-			(at 48.26 205.74 0)
+			(at 45.72 214.63 0)
 			(effects
 				(font
@@
 	)
 	(symbol
-		(lib_id "Device:LED")
-		(at 48.26 231.14 90)
-		(unit 1)
-		(exclude_from_sim no)
-		(in_bom yes)
-		(on_board yes)
-		(dnp no)
-		(fields_autoplaced yes)
-		(property "Reference" "D1"
-			(at 52.07 231.4574 90)
-			(effects
-				(font
-					(size 1.27 1.27)
-				)
-				(justify right)
-			)
-		)
-		(property "Value" "LED"
-			(at 52.07 233.9974 90)
-			(effects
-				(font
-					(size 1.27 1.27)
-				)
-				(justify right)
-			)
-		)
-		(property "Footprint" "LED_SMD:LED_0805_2012Metric_Pad1.15x1.40mm_HandSolder"
-			(at 48.26 231.14 0)
-			(effects
-				(font
-					(size 1.27 1.27)
-				)
-				(hide yes)
-			)
-		)
-		(property "Datasheet" "~"
-			(at 48.26 231.14 0)
-			(effects
-				(font
-					(size 1.27 1.27)
-				)
-				(hide yes)
-			)
-		)
-		(property "Description" "Light emitting diode"
-			(at 48.26 231.14 0)
-			(effects
-				(font
-					(size 1.27 1.27)
-				)
-				(hide yes)
-			)
-		)
-		(pin "1"
-		)
-		(pin "2"
-		)
-		(instances
-			(project ""
-				(path "/61e913ea-868b-4b77-8707-03788b798f2b"
-					(reference "D1")
-					(unit 1)
-				)
-			)
-		)
-	)
-	(symbol
 		(lib_id "Device:R")
 		(at 144.78 143.51 0)
@@
 	(symbol
 		(lib_id "power:GND")
-		(at 48.26 236.22 0)
+		(at 111.76 219.71 0)
 		(unit 1)
 		(exclude_from_sim no)
@@
 		(fields_autoplaced yes)
 		(property "Reference" "#PWR029"
-			(at 48.26 242.57 0)
+			(at 111.76 226.06 0)
 			(effects
 				(font
@@
 		)
 		(property "Value" "GND"
-			(at 50.8 237.49 0)
+			(at 114.3 220.98 0)
 			(effects
 				(font
@@
 		)
 		(property "Footprint" ""
-			(at 48.26 236.22 0)
+			(at 111.76 219.71 0)
 			(effects
 				(font
@@
 		)
 		(property "Datasheet" ""
-			(at 48.26 236.22 0)
+			(at 111.76 219.71 0)
 			(effects
 				(font
@@
 		)
 		(property "Description" ""
-			(at 48.26 236.22 0)
+			(at 111.76 219.71 0)
 			(effects
 				(font

Commit message: brake light and RTDS
Connections:
- net +12V: now also P1.C4, P1.D8; no longer U7.1
- net +3V3: now also P1.D10
- net +5V: no longer P1.D8
- net GND: now also U7.1, U7.4; no longer P1.C3, P1.C4, P1.D7, P1.D9, U7.6
- net RTDS: now also P1.D9, U7.3; no longer P1.D10, U1.CN7_23 (PC13)
- net RTDS_Signal: now reaches U7.5
- net RTDS_Signal: now also U1.CN7_23 (PC13)
- new net Brake_light: P1.C3, U7.6
- no-connect marks 53 -> 51
